File: PCB/TEMP_ctrl/TEMP_ctrl.kicad_pcb (KiCad board)
At the start: 2 copper layers, 82.2 x 52.5 mm, 38 parts, among them J1 CH1, J2 CH2, J3 CH3, J4 CH4, U1 LMC6484, U2 102010388, U3 AP2112K-3.3, U4 LMC6484

Commit message: pc: working on the PCB
Parts:
- added Q3: DMN2056U, Package_TO_SOT_SMD:SOT-23, F.Cu at (149.6, 100.7)
- added R18: 10kΩ, PCM_JLCPCB:R_1206, F.Cu at (146.2, 100.2)
- moved J1 2.74 mm to (158.6, 93.2), turned to 180 degrees
- moved J2 2.55 mm to (177.2, 93.2), turned to 180 degrees
- moved J3 2.55 mm to (167.9, 93.2), turned to 180 degrees
- moved J4 2.55 mm to (186.5, 93.2), turned to 180 degrees
- moved R16 0.25 mm to (178.3, 105.5)
- moved R17 0.25 mm to (187.7, 105.5)
- moved R4 0.25 mm to (159.7, 105.5)
- moved R9 0.25 mm to (169.0, 105.5)
Connections:
- C11 pad 1: Net-(J2-Pin_2) -> Net-(J2-Pin_1)
- C12 pad 1: Net-(J4-Pin_2) -> Net-(J4-Pin_1)
- C13 pad 1: Net-(J1-Pin_2) -> Net-(J1-Pin_1)
- C14 pad 1: Net-(J3-Pin_2) -> Net-(J3-Pin_1)
- J1 pad 1: VAA -> Net-(J1-Pin_1)
- J1 pad 2: Net-(J1-Pin_2) -> VAA
- J2 pad 1: VAA -> Net-(J2-Pin_1)
- J2 pad 2: Net-(J2-Pin_2) -> VAA
- J3 pad 1: VAA -> Net-(J3-Pin_1)
- J3 pad 2: Net-(J3-Pin_2) -> VAA
- J4 pad 1: VAA -> Net-(J4-Pin_1)
- J4 pad 2: Net-(J4-Pin_2) -> VAA
- R11 pad 1: Net-(J2-Pin_2) -> Net-(J2-Pin_1)
- R11 pad 2: GNDA -> R_COM
- R12 pad 1: Net-(J4-Pin_2) -> Net-(J4-Pin_1)
- R12 pad 2: GNDA -> R_COM
- R13 pad 1: Net-(J2-Pin_2) -> Net-(J2-Pin_1)
- R14 pad 1: Net-(J4-Pin_2) -> Net-(J4-Pin_1)
- R2 pad 1: Net-(J1-Pin_2) -> Net-(J1-Pin_1)
- R2 pad 2: GNDA -> R_COM
- R3 pad 1: Net-(J1-Pin_2) -> Net-(J1-Pin_1)
- R7 pad 1: Net-(J3-Pin_2) -> Net-(J3-Pin_1)
- R7 pad 2: GNDA -> R_COM
- R8 pad 1: Net-(J3-Pin_2) -> Net-(J3-Pin_1)
- U2 pad 7: unconnected-(U2-PB08_A6_D6_TX-Pad7) -> R_PWR_EN
Routing:
- net R_COM: track 0.00 -> 38.3 mm, vias 0 -> 4
- net R_PWR_EN: track 0.00 -> 27.1 mm, vias 0 -> 1
- net Net-(J4-Pin_2): track 9.34 -> 0.00 mm
- net Net-(J4-Pin_1): track 0.00 -> 9.34 mm
- net Net-(J2-Pin_2): track 9.32 -> 0.00 mm
- net Net-(J2-Pin_1): track 0.00 -> 9.32 mm
- net Net-(J1-Pin_2): track 9.31 -> 0.00 mm
- net Net-(J1-Pin_1): track 0.00 -> 9.31 mm
- net Net-(J3-Pin_2): track 9.31 -> 0.00 mm
- net Net-(J3-Pin_1): track 0.00 -> 9.31 mm
- net VAA/2: track 59.4 -> 58.1 mm
- net VAA: track 96.8 -> 97.6 mm
- net Net-(U1A--): track 9.38 -> 10.1 mm
- net Net-(U4A--): track 9.29 -> 9.95 mm
- net GNDA: vias 313 -> 263
Other:
- board text added: "Temp_mon&ctrl FZ. Liu Apr, 2025"

Commit message: mac: finished PCB design
Parts:
- added C15: 10nF, PCM_JLCPCB:C_1206, F.Cu at (148.1, 101.7)
- added G***: LOGO, LOGO, F.Cu at (185.1, 134.0)
- added J10: Heater3, TerminalBlock:TerminalBlock_MaiXu_MX126-5.0-02P_1x02_P5.00mm, F.Cu at (114.7, 116.8)
- added J11: Heater2, TerminalBlock:TerminalBlock_MaiXu_MX126-5.0-02P_1x02_P5.00mm, F.Cu at (114.7, 105.2)
- added J12: Heater4, TerminalBlock:TerminalBlock_MaiXu_MX126-5.0-02P_1x02_P5.00mm, F.Cu at (114.7, 128.5)
- added J5: Conn_01x01_Pin, TestPoint:TestPoint_Pad_4.0x4.0mm, B.Cu at (117.5, 138.9)
- added J6: Conn_01x01_Pin, TestPoint:TestPoint_Pad_4.0x4.0mm, F.Cu at (122.6, 137.6)
- added J7: LCD, Connector_PinHeader_2.54mm:PinHeader_1x04_P2.54mm_Vertical, F.Cu at (136.3, 102.9)
- added J9: Heater1, TerminalBlock:TerminalBlock_MaiXu_MX126-5.0-02P_1x02_P5.00mm, F.Cu at (114.7, 93.5)
- added Q1: IRLZ44N, Package_TO_SOT_THT:TO-220-3_Vertical, F.Cu at (126.9, 109.3)
- added Q2: IRLZ44N, Package_TO_SOT_THT:TO-220-3_Vertical, F.Cu at (126.9, 98.2)
- added Q4: IRLZ44N, Package_TO_SOT_THT:TO-220-3_Vertical, F.Cu at (126.9, 120.4)
- added Q5: IRLZ44N, Package_TO_SOT_THT:TO-220-3_Vertical, F.Cu at (126.9, 131.5)
- added R15: 0Ω, PCM_JLCPCB:R_1206, F.Cu at (128.3, 135.5)
- added R19: 100Ω, PCM_JLCPCB:R_1206, F.Cu at (133.4, 123.6)
- added R20: 100Ω, PCM_JLCPCB:R_1206, F.Cu at (133.4, 126.2)
- added R21: 100Ω, PCM_JLCPCB:R_1206, F.Cu at (133.4, 128.7)
- added R22: 100Ω, PCM_JLCPCB:R_1206, F.Cu at (133.4, 131.2)
- added R23: 10kΩ, PCM_JLCPCB:R_1206, F.Cu at (129.7, 99.6)
- added R24: 10kΩ, PCM_JLCPCB:R_1206, F.Cu at (129.7, 121.8)
- added R25: 10kΩ, PCM_JLCPCB:R_1206, F.Cu at (129.7, 130.0)
- added R26: 10kΩ, PCM_JLCPCB:R_1206, F.Cu at (129.7, 110.7)
- added R27: 10kΩ, PCM_JLCPCB:R_1206, F.Cu at (148.2, 126.2)
- added R28: 10kΩ, PCM_JLCPCB:R_1206, F.Cu at (148.2, 128.7)
- moved Q3 2.23 mm to (149.9, 98.5)
- moved R18 2.06 mm to (146.6, 98.2)
Connections:
- U2 pad 10: unconnected-(U2-PA5_A9_D9_MISO-Pad10) -> HEATER3
- U2 pad 11: unconnected-(U2-PA6_A10_D10_MOSI-Pad11) -> HEATER4
- U2 pad 12: unconnected-(U2-3V3-Pad12) -> +3.3V
- U2 pad 5: unconnected-(U2-PA8_A4_D4_SDA-Pad5) -> SDA
- U2 pad 6: unconnected-(U2-PA9_A5_D5_SCL-Pad6) -> SCL
- U2 pad 8: unconnected-(U2-PB09_A7_D7_RX-Pad8) -> HEATER1
- U2 pad 9: unconnected-(U2-PA7_A8_D8_SCK-Pad9) -> HEATER2
Routing:
- net +3.3V: track 0.00 -> 47.2 mm, vias 0 -> 1
- net SCL: track 0.00 -> 35.4 mm
- net SDA: track 0.00 -> 35.2 mm
- net Net-(Q2-G): track 0.00 -> 29.5 mm, vias 0 -> 2
- net Net-(Q1-G): track 0.00 -> 20.6 mm, vias 0 -> 2
- net Net-(J9-Pin_1): track 0.00 -> 13.1 mm
- net Net-(J11-Pin_1): track 0.00 -> 12.8 mm
- net Net-(J10-Pin_1): track 0.00 -> 12.6 mm
- net Net-(J12-Pin_1): track 0.00 -> 12.4 mm
- net Net-(Q4-G): track 0.00 -> 12.1 mm, vias 0 -> 2
- net R_PWR_EN: track 27.1 -> 38.3 mm
- net Net-(Q5-G): track 0.00 -> 5.14 mm
- net HEATER4: track 0.00 -> 2.81 mm
- net HEATER3: track 0.00 -> 2.81 mm
- net HEATER2: track 0.00 -> 2.81 mm
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- added copper zone on B.Cu, net +24V
- added copper zone on B.Cu, net GNDPWR
- added copper zone on F.Cu, net GNDPWR
Other:
- board text added: "HEATER #1"
- board text added: "HEATER #2"
- board text added: "HEATER #3"
- board text added: "HEATER #4"
- board text added: "RTD #1"
- board text added: "RTD #2"
- board text added: "RTD #3"
- board text added: "RTD #4"

Commit message: pc: working on the PCB
Parts:
- moved C15 4.89 mm to (143.2, 102.0), turned to 180 degrees
- moved R18 3.73 mm to (143.3, 99.8), turned to 0 degrees
- moved Q3 2.27 mm to (147.7, 98.8)
- moved J6 0.90 mm to (122.6, 138.5)
- moved J5 0.38 mm to (117.5, 138.5)
Connections:
- C15 pad 2: GNDA -> GNDD
- R18 pad 1: R_PWR_EN -> GNDD
- R18 pad 2: GNDA -> R_PWR_EN
Routing:
- net R_COM: track 38.9 -> 41.0 mm
- net R_PWR_EN: track 38.3 -> 37.0 mm
- net GNDD: vias 22 -> 23
- net GNDA: vias 234 -> 241
- net CH1: vias 1 -> 0
