File: PCB/TEMP_ctrl_DS18B20/TEMP_ctrl_DS18B20.kicad_pcb (KiCad board)
At the start: 2 copper layers, 61.8 x 76 mm, 45 parts, among them J1 Heater2, J10 Heater3, J11 Heater2, J12 Heater4, J2 Heater4, J5 Conn_01x01_Pin, J6 Conn_01x01_Pin, J7 LCD, J9 Heater1, Q1 IRLZ44N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

Commit message: PC: working on the DS18B20 PCB design
Parts:
- added J13: 691412320003, Mylib:691412320003, F.Cu at (155.2, 102.0)
- added J14: 691412320003, Mylib:691412320003, F.Cu at (155.2, 88.3)
- added J15: 691412320003, Mylib:691412320003, F.Cu at (155.2, 74.6)
- added J16: 691412320003, Mylib:691412320003, F.Cu at (140.6, 102.0)
- added J17: 691412320003, Mylib:691412320003, F.Cu at (140.6, 88.3)
- added J18: 691412320003, Mylib:691412320003, F.Cu at (140.6, 74.6)
- added J3: 691412320002, Mylib:691412320002, F.Cu at (112.5, 95.4)
- added J4: 691412320002, Mylib:691412320002, F.Cu at (112.5, 107.1)
- added J8: 691412320002, Mylib:691412320002, F.Cu at (112.5, 72.0)
- added R1: 4.7kΩ, PCM_JLCPCB:R_1206, F.Cu at (142.1, 110.0)
- J1: value Heater2 -> 691412320002; footprint TerminalBlock:TerminalBlock_MaiXu_MX126-5.0-02P_1x02_P5.00mm -> Mylib:691412320002
- J10: value Heater3 -> 691412320003; footprint TerminalBlock:TerminalBlock_MaiXu_MX126-5.0-02P_1x02_P5.00mm -> Mylib:691412320003
- J11: value Heater2 -> 691412320003; footprint TerminalBlock:TerminalBlock_MaiXu_MX126-5.0-02P_1x02_P5.00mm -> Mylib:691412320003
- J12: value Heater4 -> 691412320003; footprint TerminalBlock:TerminalBlock_MaiXu_MX126-5.0-02P_1x02_P5.00mm -> Mylib:691412320003
- J2: value Heater4 -> 691412320002; footprint TerminalBlock:TerminalBlock_MaiXu_MX126-5.0-02P_1x02_P5.00mm -> Mylib:691412320002
- J9: value Heater1 -> 691412320002; footprint TerminalBlock:TerminalBlock_MaiXu_MX126-5.0-02P_1x02_P5.00mm -> Mylib:691412320002
- moved J12 77.1 mm to (169.9, 74.6), turned to 180 degrees
- moved J11 57.7 mm to (169.9, 88.3), turned to 180 degrees
- moved J10 57.1 mm to (169.9, 102.0), turned to 180 degrees
- moved J2 49.1 mm to (112.5, 130.8)
- moved J1 48.7 mm to (112.5, 118.7)
- moved R2 42.1 mm to (132.1, 76.4), turned to 90 degrees
- moved R4 33.0 mm to (132.1, 88.1), turned to 90 degrees
- moved R27 29.2 mm to (170.9, 124.4)
- moved R28 29.2 mm to (170.9, 127.0)
- moved R19 24.0 mm to (132.1, 99.6), turned to 90 degrees
- moved J7 19.9 mm to (167.7, 130.8), turned to 90 degrees
- moved C3 18.3 mm to (153.9, 131.6)
- moved R20 15.5 mm to (132.1, 110.7), turned to 90 degrees
- moved C2 12.2 mm to (143.2, 128.3), turned to 180 degrees
- moved J9 10.0 mm to (112.5, 83.7)
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Connections:
- C22 pad 2: GND -> GNDD
- C23 pad 1: GND -> GNDD
- C24 pad 1: GND -> GNDD
- C26 pad 2: GND -> GNDD
- J1 pad 1: Net-(J1-Pin_1) -> +24V
- J1 pad 2: +24V -> Net-(Q4-D)
- J10 pad 1: Net-(J10-Pin_1) -> GNDD
- J10 pad 2: +24V -> DS_D
- J11 pad 1: Net-(J11-Pin_1) -> GNDD
- J11 pad 2: +24V -> DS_D
- J12 pad 1: Net-(J12-Pin_1) -> GNDD
- J12 pad 2: +24V -> DS_D
- J2 pad 1: Net-(J2-Pin_1) -> +24V
- J2 pad 2: +24V -> Net-(Q5-D)
- J9 pad 1: Net-(J9-Pin_1) -> +24V
- J9 pad 2: +24V -> Net-(Q6-D)
- Q1 pad 2: Net-(J11-Pin_1) -> Net-(Q1-D)
- Q2 pad 2: Net-(J9-Pin_1) -> Net-(Q2-D)
- Q3 pad 2: Net-(J1-Pin_1) -> Net-(Q3-D)
- Q4 pad 2: Net-(J10-Pin_1) -> Net-(Q4-D)
- Q5 pad 2: Net-(J12-Pin_1) -> Net-(Q5-D)
- Q6 pad 2: Net-(J2-Pin_1) -> Net-(Q6-D)
- Y3 pad 2: GND -> GNDD
- Y3 pad 4: GND -> GNDD
Routing:
- net DS_D: track 0.00 -> 116.9 mm
- net +3.3V: track 0.00 -> 115.3 mm
- net Net-(Q3-G): track 47.3 -> 2.79 mm, vias 2 -> 0
- net Net-(Q6-G): track 38.1 -> 2.79 mm, vias 2 -> 0
- net Net-(Q2-G): track 29.2 -> 2.80 mm, vias 2 -> 0
- net Net-(Q1-G): track 20.6 -> 2.80 mm, vias 2 -> 0
- net VAA: track 2.18 -> 17.9 mm
- net Net-(J2-Pin_1): track 13.1 -> 0.00 mm
- net Net-(J1-Pin_1): track 13.1 -> 0.00 mm
- net Net-(J9-Pin_1): track 13.1 -> 0.00 mm
- net Net-(Q6-D): track 0.00 -> 12.8 mm
- net Net-(Q3-D): track 0.00 -> 12.8 mm
- net Net-(J11-Pin_1): track 12.8 -> 0.00 mm
- net Net-(Q2-D): track 0.00 -> 12.8 mm
- net Net-(J10-Pin_1): track 12.6 -> 0.00 mm
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Other:
- board size 61.8 x 76 mm -> 74 x 76 mm
- board text added: "DATA"
- board text added: "DS1"
- board text added: "DS2"
- board text added: "DS3"
- board text added: "DS4"
- board text added: "DS5"
- board text added: "DS6"
- board text added: "DS7"
- board text added: "DS8"
- board text added: "DS9"
- board text added: "GND"
- board text added: "VDD"

Commit message: PC: working on the DS18B20 PCB design
Parts:
- moved R27 15.7 mm to (159.5, 135.2), turned to -90 degrees
- moved R28 12.1 mm to (162.1, 135.2), turned to -90 degrees
- moved R15 1.78 mm to (128.3, 137.3)
- moved C1 1.70 mm to (153.1, 136.1)
- moved U3 1.70 mm to (149.8, 135.6)
- moved C10 1.70 mm to (146.2, 135.4)
- moved C5 1.41 mm to (155.8, 121.2)
- moved J7 0.81 mm to (167.5, 131.6)
- moved C4 0.49 mm to (143.2, 126.8)
- moved J6 0.39 mm to (122.1, 138.7)
- moved J5 0.37 mm to (117.2, 138.7)
Connections:
- C1 pad 1: VAA -> +3.3V
- C2 pad 1: VAA -> +3.3V
- C3 pad 1: VAA -> +3.3V
- C4 pad 1: VAA -> +3.3V
- C5 pad 1: VAA -> +3.3V
- C6 pad 1: VAA -> +3.3V
- R19 pad 1: HEATER1 -> HEATER3
- R2 pad 1: HEATER2 -> HEATER1
- R20 pad 1: HEATER2 -> HEATER4
- R21 pad 1: HEATER3 -> HEATER5
- R22 pad 1: HEATER4 -> HEATER6
- R4 pad 1: HEATER4 -> HEATER2
- U1 pad 1: VAA -> +3.3V
- U1 pad 12: unconnected-(U1-PA4-Pad12) -> DS_D
- U1 pad 13: unconnected-(U1-PA5-Pad13) -> HEATER1
- U1 pad 14: unconnected-(U1-PA6-Pad14) -> HEATER2
- U1 pad 15: unconnected-(U1-PA7-Pad15) -> HEATER3
- U1 pad 16: unconnected-(U1-PB0-Pad16) -> HEATER4
- U1 pad 17: unconnected-(U1-PB1-Pad17) -> HEATER5
- U1 pad 18: unconnected-(U1-PB2-Pad18) -> HEATER6
- U1 pad 20: VAA -> +3.3V
- U1 pad 21: VAA -> +3.3V
- U1 pad 24: VAA -> +3.3V
- U1 pad 36: VAA -> +3.3V
- U1 pad 48: VAA -> +3.3V
- U3 pad 5: VAA -> +3.3V
Routing:
- net +3.3V: track 115.3 -> 212.0 mm, vias 0 -> 5
- net HEATER1: track 0.00 -> 53.0 mm
- net HEATER2: track 0.00 -> 41.9 mm
- net HEATER3: track 0.00 -> 31.0 mm
- net HEATER4: track 0.00 -> 20.5 mm
- net VAA: track 17.9 -> 0.00 mm
- net HEATER6: track 0.00 -> 16.5 mm
- net HEATER5: track 0.00 -> 14.7 mm
- net DS_D: track 116.9 -> 131.2 mm
- net SCL: track 0.00 -> 13.3 mm
- net SDA: track 0.00 -> 11.3 mm
- net unconnected-(U1-PB7-Pad44): track 0.00 -> 10.9 mm
- net unconnected-(U1-PB6-Pad43): track 0.00 -> 10.8 mm
- net unconnected-(U1-PB5-Pad42): track 0.00 -> 10.7 mm
- net unconnected-(U1-PB4-Pad41): track 0.00 -> 10.7 mm
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
Commit message: PC: working on the DS18B20 PCB design
Parts:
- added C7: 10uF, PCM_JLCPCB:C_1206, F.Cu at (135.8, 134.3)
- added D1: LED_Small_Filled, LED_SMD:LED_1206_3216Metric, F.Cu at (135.9, 131.8)
- added D2: LED_Small_Filled, LED_SMD:LED_1206_3216Metric, F.Cu at (151.5, 139.3)
- added J19: Conn_01x04_Pin, Connector_PinHeader_2.54mm:PinHeader_1x04_P2.54mm_Vertical, F.Cu at (167.5, 127.5)
- added J20: Conn_01x04_Pin, Connector_PinHeader_2.54mm:PinHeader_1x04_P2.54mm_Vertical, F.Cu at (167.5, 123.8)
- added J21: Conn_01x04_Pin, Connector_PinHeader_2.54mm:PinHeader_1x04_P2.54mm_Vertical, F.Cu at (167.5, 120.2)
- added J22: USB_B_Micro, Connector_USB:USB_Micro-B_Amphenol_10104110_Horizontal, F.Cu at (138.8, 138.7)
- added J23: Conn_01x04_Pin, Connector_PinHeader_2.54mm:PinHeader_1x04_P2.54mm_Vertical, F.Cu at (155.6, 139.3)
- added R6: 1kΩ, PCM_JLCPCB:R_1206, F.Cu at (135.8, 129.5)
- added R7: 1kΩ, PCM_JLCPCB:R_1206, F.Cu at (146.8, 139.3)
- moved J8 2.25 mm to (112.5, 74.3)
- moved J9 2.25 mm to (112.5, 86.0)
- moved J3 2.09 mm to (112.5, 97.5)
- moved J4 1.55 mm to (112.5, 108.6)
- moved R27 1.47 mm to (159.4, 133.7)
- moved R28 1.47 mm to (162.0, 133.7)
- moved C1 1.36 mm to (153.1, 134.7)
- moved J1 1.00 mm to (112.5, 119.7)
- moved J7 0.44 mm to (167.5, 131.2)
- moved C10 0.23 mm to (146.2, 135.2)
- moved U3 0.23 mm to (149.8, 135.3)
Connections:
- U1 pad 33: unconnected-(U1-PA11-Pad33) -> USB-
- U1 pad 34: unconnected-(U1-PA12-Pad34) -> USB+
- U1 pad 37: unconnected-(U1-PA13-Pad37) -> SWDIO
- U1 pad 38: unconnected-(U1-PA14-Pad38) -> SWDCLK
Routing:
- net USB-: track 0.00 -> 17.9 mm
- net USB+: track 0.00 -> 17.8 mm
- net SWDCLK: track 0.00 -> 15.2 mm, vias 0 -> 1
- net SWDIO: track 0.00 -> 13.4 mm, vias 0 -> 1
- net +5V: track 5.36 -> 17.1 mm, vias 0 -> 2
- net unconnected-(J21-Pin_4-Pad4): track 0.00 -> 10.2 mm
- net unconnected-(U1-PA14-Pad38): track 9.40 -> 0.00 mm
- net unconnected-(J21-Pin_3-Pad3): track 0.00 -> 8.50 mm
- net unconnected-(U1-PA13-Pad37): track 8.23 -> 0.00 mm
- net +3.3V: track 212.0 -> 218.1 mm
- net unconnected-(J21-Pin_2-Pad2): track 0.00 -> 5.87 mm
- net unconnected-(J21-Pin_1-Pad1): track 0.00 -> 2.59 mm
- net Net-(D1-K): track 0.00 -> 2.38 mm
- net Net-(D2-K): track 0.00 -> 1.81 mm
- net SCL: track 13.3 -> 12.3 mm
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Other:
- board text added: "CL"
- board text added: "DA"
- board text added: "G"
- board text added: "IO"
- board text added: "V"

Commit message: PC: finished DS18B20 PCB design
Parts:
- added G***: LOGO, LOGO, F.Cu at (112.2, 139.4)
Connections:
- J19 pad 1: unconnected-(J19-Pin_1-Pad1) -> PB3
- J19 pad 2: unconnected-(J19-Pin_2-Pad2) -> PA15
- J19 pad 3: unconnected-(J19-Pin_3-Pad3) -> GNDD
- J19 pad 4: unconnected-(J19-Pin_4-Pad4) -> GNDD
- J20 pad 1: unconnected-(J20-Pin_1-Pad1) -> PB7
- J20 pad 2: unconnected-(J20-Pin_2-Pad2) -> PB6
- J20 pad 3: unconnected-(J20-Pin_3-Pad3) -> PB5
- J20 pad 4: unconnected-(J20-Pin_4-Pad4) -> PB4
- J21 pad 1: unconnected-(J21-Pin_1-Pad1) -> PB9
- J21 pad 2: unconnected-(J21-Pin_2-Pad2) -> PB8
- J21 pad 3: unconnected-(J21-Pin_3-Pad3) -> PA9
- J21 pad 4: unconnected-(J21-Pin_4-Pad4) -> PA10
- U1 pad 31: unconnected-(U1-PA9-Pad31) -> PA9
- U1 pad 32: unconnected-(U1-PA10-Pad32) -> PA10
- U1 pad 39: unconnected-(U1-PA15-Pad39) -> PA15
- U1 pad 40: unconnected-(U1-PB3-Pad40) -> PB3
- U1 pad 41: unconnected-(U1-PB4-Pad41) -> PB4
- U1 pad 42: unconnected-(U1-PB5-Pad42) -> PB5
- U1 pad 43: unconnected-(U1-PB6-Pad43) -> PB6
- U1 pad 44: unconnected-(U1-PB7-Pad44) -> PB7
- U1 pad 45: unconnected-(U1-PB8-Pad45) -> PB8
- U1 pad 46: unconnected-(U1-PB9-Pad46) -> PB9
Routing:
- net PA10: track 0.00 -> 29.8 mm, vias 0 -> 1
- net PA9: track 0.00 -> 28.0 mm, vias 0 -> 1
- net PB4: track 0.00 -> 21.6 mm, vias 0 -> 1
- net PB5: track 0.00 -> 18.8 mm, vias 0 -> 1
- net PB8: track 0.00 -> 17.2 mm
- net PA15: track 0.00 -> 16.8 mm
- net PB6: track 0.00 -> 16.1 mm
- net PB9: track 0.00 -> 14.4 mm
- net PB3: track 0.00 -> 14.2 mm
- net PB7: track 0.00 -> 13.3 mm
- net unconnected-(U1-PB7-Pad44): track 10.9 -> 0.00 mm
- net unconnected-(U1-PB6-Pad43): track 10.8 -> 0.00 mm
- net unconnected-(U1-PB5-Pad42): track 10.7 -> 0.00 mm
- net unconnected-(U1-PB4-Pad41): track 10.7 -> 0.00 mm
- net unconnected-(U1-PB8-Pad45): track 10.5 -> 0.00 mm
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