File: PCB/TEMP_ctrl_DS18B20/TEMP_ctrl_DS18B20.kicad_sch (KiCad schematic)
At the start: 45 parts, among them J1 Heater2, J10 Heater3, J11 Heater2, J12 Heater4, J2 Heater4, J5 Conn_01x01_Pin, J6 Conn_01x01_Pin, J7 LCD, J9 Heater1, Q1 IRLZ44N, Q2 IRLZ44N, Q3 IRLZ44N, Q4 IRLZ44N, Q5 IRLZ44N, Q6 IRLZ44N, U1 STM32G431CBTx, U3 AP2112K-3.3, Y2 32KHz, Y3 ECS-160-12-33-AGN-TR3

Commit message: PC: working on the DS18B20 PCB design
Parts:
- removed J1, J11: Heater2, TerminalBlock:TerminalBlock_MaiXu_MX126-5.0-02P_1x02_P5.00mm, symbol Connector:Screw_Terminal_01x02
- removed J10: Heater3, TerminalBlock:TerminalBlock_MaiXu_MX126-5.0-02P_1x02_P5.00mm, symbol Connector:Screw_Terminal_01x02
- removed J12, J2: Heater4, TerminalBlock:TerminalBlock_MaiXu_MX126-5.0-02P_1x02_P5.00mm, symbol Connector:Screw_Terminal_01x02
- removed J9: Heater1, TerminalBlock:TerminalBlock_MaiXu_MX126-5.0-02P_1x02_P5.00mm, symbol Connector:Screw_Terminal_01x02
- added J1, J2, J3, J4, J8, J9: 691412320002, Mylib:691412320002, symbol 691412320002:691412320002
- added J10, J11, J12, J13, J14, J15, J16, J17, J18: 691412320003, Mylib:691412320003, symbol 691412320003:691412320003
- added R1: 4.7kΩ, PCM_JLCPCB:R_1206, symbol PCM_JLCPCB-Resistors:1206,1kΩ
Connections:
- net GND is gone; now on net GNDD: C22.2, C23.1, C24.1, C26.2, Y3.2 (GND_1), Y3.4 (GND_2)
- net +24V: now also J1.1, J2.1, J3.1, J4.1, J8.1, J9.1
- net +3.3V: now also J10.3, J11.3, J12.3, J13.3, J14.3, J15.3, J16.3, J17.3, J18.3, R1.2
- net GNDD: now also J10.1, J11.1, J12.1, J13.1, J14.1, J15.1, J16.1, J17.1, J18.1
- net at Q2.2 (D): now also J3.2
- net at Q6.2 (D): now also J9.2
- net at Q5.2 (D): now also J2.2
- net at Q3.2 (D): now also J8.2
- net at Q4.2 (D): now also J1.2
- net at Q1.2 (D): now also J4.2
- new net DS_D: J10.2, J11.2, J12.2, J13.2, J14.2, J15.2, J16.2, J17.2, J18.2, R1.1
Other:
- moved on the sheet: C1, C10, C22, C26, U3, Y3

Commit message: PC: working on the DS18B20 PCB design
Connections:
- net VAA is gone; now on net +3.3V: C1.1, C2.1, C3.1, C4.1, C5.1, C6.1, U1.1 (VBAT), U1.20 (VREF+), U1.21 (VDDA), U1.24 (VDD), U1.36 (VDD), U1.48 (VDD), U3.5 (VOUT)
- net DS_D: now also U1.12 (PA4)
- net HEATER1: now also R2.1, U1.13 (PA5); no longer R19.1
- net HEATER2: now also R4.1, U1.14 (PA6); no longer R2.1, R20.1
- net HEATER3: now also R19.1, U1.15 (PA7); no longer R21.1
- net HEATER4: now also R20.1, U1.16 (PB0); no longer R22.1, R4.1
- net HEATER5: now reaches U1.17 (PB1)
- net HEATER5: now also R21.1
- net HEATER6: now reaches U1.18 (PB2)
- net HEATER6: now also R22.1

Commit message: PC: working on the DS18B20 PCB design
Parts:
- added C7: 10uF, PCM_JLCPCB:C_1206, symbol PCM_JLCPCB-Capacitors:1206,100nF
- added D1, D2: LED_Small_Filled, LED_SMD:LED_1206_3216Metric, symbol Device:LED_Small_Filled
- added J19, J20, J21, J23: Conn_01x04_Pin, Connector_PinHeader_2.54mm:PinHeader_1x04_P2.54mm_Vertical, symbol Connector:Conn_01x04_Pin
- added J22: USB_B_Micro, Connector_USB:USB_Micro-B_Amphenol_10104110_Horizontal, symbol Connector:USB_B_Micro
- added R6, R7: 1kΩ, PCM_JLCPCB:R_1206, symbol PCM_JLCPCB-Resistors:1206,1kΩ
Connections:
- net +3.3V: now also D2.2 (A), J23.1 (Pin_1)
- net +5V: now also C7.1, D1.2 (A), J22.1 (VBUS)
- net GNDD: now also C7.2, J22.5 (GND), J22.6 (Shield), J23.4 (Pin_4), R6.1, R7.1
- net USB-: now reaches U1.33 (PA11)
- net USB-: now also J22.2 (D-)
- net USB+: now reaches U1.34 (PA12)
- net USB+: now also J22.3 (D+)
- net SWDIO: now reaches U1.37 (PA13)
- net SWDIO: now also J23.2 (Pin_2)
- net SWDCLK: now reaches U1.38 (PA14)
- net SWDCLK: now also J23.3 (Pin_3)
- new net: D1.1 (K), R6.2
- new net: D2.1 (K), R7.2
- no-connect marks 0 -> 1
Other:
- note added: "Extension connectors"
- moved on the sheet: J7, R1, R27, R28

Commit message: PC: finished DS18B20 PCB design
Connections:
- net GNDD: now also J19.3 (Pin_3), J19.4 (Pin_4)
- net PB3: now reaches J19.1 (Pin_1)
- net PB3: now also U1.40 (PB3)
- net PA15: now reaches J19.2 (Pin_2)
- net PA15: now also U1.39 (PA15)
- net PB9: now reaches J21.1 (Pin_1)
- net PB9: now also U1.46 (PB9)
- net PB8: now reaches J21.2 (Pin_2)
- net PB8: now also U1.45 (PB8)
- net PA9: now reaches J21.3 (Pin_3)
- net PA9: now also U1.31 (PA9)
- net PA10: now reaches J21.4 (Pin_4)
- net PA10: now also U1.32 (PA10)
- net PB7: now reaches J20.1 (Pin_1)
- net PB7: now also U1.44 (PB7)
- net PB6: now reaches J20.2 (Pin_2)
- net PB6: now also U1.43 (PB6)
- net PB5: now reaches J20.3 (Pin_3)
- net PB5: now also U1.42 (PB5)
- net PB4: now reaches J20.4 (Pin_4)
- net PB4: now also U1.41 (PB4)
